File: ESP32-game-console.kicad_pcb (KiCad board)
At the start: 2 copper layers, 100 x 50 mm, 68 parts, among them J1 USB_C_Receptacle_USB2.0_16P, J2 Micro_SD_Card, J3 BAT+, J4 BAT-, SW1 LEFT, SW10 B, SW11 L, SW12 R, SW18 SELECT, SW19 START, SW2 RIGHT, SW3 SW_DPST_x2, SW7 UP, SW8 DOWN, SW9 A, U1 ESP32-S3-WROOM-1, U2 USBLC6-2SC6, U3 LF33_TO252, U4 TP4056-42-ESOP8, U6 PAM8403D

Commit message: Detaylar
Routing:
- net /Screen_DC: track 23.7 -> 21.0 mm
- net Net-(U1-IO0): track 35.4 -> 37.1 mm
- net +3.3V: track 256.1 -> 257.7 mm
- net /D+: track 10.2 -> 9.07 mm
- net /D-: track 6.93 -> 7.52 mm

Commit message: Detaylar2
Routing:
- net +5V: track 75.7 -> 79.1 mm
- net /Screen_DC: track 21.0 -> 23.7 mm
- net GND: vias 39 -> 41
Changed lines of the file:
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@@
 	)
 	(setup
+		(stackup
+			(layer "F.SilkS"
+				(type "Top Silk Screen")
+			)
+			(layer "F.Paste"
+				(type "Top Solder Paste")
+			)
+			(layer "F.Mask"
+				(type "Top Solder Mask")
+				(thickness 0.01)
+			)
+			(layer "F.Cu"
+				(type "copper")
+				(thickness 0.035)
+			)
+			(layer "dielectric 1"
+				(type "core")
+				(thickness 1.51)
+				(material "FR4")
+				(epsilon_r 4.5)
+				(loss_tangent 0.02)
+			)
+			(layer "B.Cu"
+				(type "copper")
+				(thickness 0.035)
+			)
+			(layer "B.Mask"
+				(type "Bottom Solder Mask")
+				(thickness 0.01)
+			)
+			(layer "B.Paste"
+				(type "Bottom Solder Paste")
+			)
+			(layer "B.SilkS"
+				(type "Bottom Silk Screen")
+			)
+			(copper_finish "None")
+			(dielectric_constraints no)
+		)
 		(pad_to_mask_clearance 0)
 		(allow_soldermask_bridges_in_footprints no)
@@
 		(capping no)
 		(filling no)
+		(zone_defaults)
 		(pcbplotparams
 			(layerselection 0x00000000_00000000_55555555_5755f5ff)
@@
 	)
 	(gr_text "https://github.com/EnesOzdmir\n	/ESP-micro-GAMEBOY"
-		(at 135.68 123.95 0)
+		(at 135.72 124.34 0)
 		(layer "B.SilkS")
 		(effects
 			(font
-				(size 0.5 0.5)
+				(size 0.8 0.5)
 				(thickness 0.125)
 				(bold yes)
@@
 	)
 	(via
+		(at 174.27 86.05)
+		(size 0.6)
+		(drill 0.3)
+		(layers "F.Cu" "B.Cu")
+		(net "GND")
+	)
+	(via
 		(at 172.045491 100.730542)
 		(size 0.6)
@@
 	)
 	(via
+		(at 116.02 85.53)
+		(size 0.6)
+		(drill 0.3)
+		(layers "F.Cu" "B.Cu")
+		(free yes)
+		(net "GND")
+	)
+	(via
 		(at 177.93 116.63)
 		(size 0.6)
@@
 	)
 	(segment
-		(start 165.300456 88.04)
-		(end 165.645 87.695456)
+		(start 165.18 87.680456)
+		(end 165.18 87.82)
 		(width 0.3)
 		(layer "F.Cu")
@@
 	)
 	(segment
-		(start 164.96 88.04)
-		(end 165.300456 88.04)
+		(start 164.96 87.355)
+		(end 164.195 86.59)
 		(width 0.3)
 		(layer "F.Cu")
@@
 	(segment
 		(start 170.47 82.390456)
-		(end 170.47 80.78)
+		(end 165.18 87.680456)
 		(width 0.3)
 		(layer "F.Cu")
@@
 	)
 	(segment
+		(start 165.18 87.575)
+		(end 164.195 86.59)
+		(width 0.3)
+		(layer "F.Cu")
+		(net "+5V")
+	)
+	(segment
 		(start 159.755 92.085)
 		(end 160.775456 92.085)
@@
 	)
 	(segment
-		(start 165.645 87.695456)
-		(end 165.645 87.215456)
+		(start 170.47 80.78)
+		(end 170.47 82.390456)
+		(width 0.3)
+		(layer "F.Cu")
+		(net "+5V")
+	)
+	(segment
+		(start 165.18 87.82)
+		(end 164.96 88.04)
 		(width 0.3)
 		(layer "F.Cu")
@@
 	)
 	(segment
-		(start 165.645 87.215456)
-		(end 170.47 82.390456)
+		(start 164.96 88.04)
+		(end 164.96 87.355)
 		(width 0.3)
 		(layer "F.Cu")
@@
 	)
 	(segment
+		(start 165.18 87.680456)
+		(end 165.18 87.575)
+		(width 0.3)
+		(layer "F.Cu")
+		(net "+5V")
+	)
+	(segment
 		(start 160.876675 91.983781)
 		(end 161.016219 91.983781)
@@
 		(net "+5V")
 	)
+	(segment
+		(start 164.195 86.59)
+		(end 164.195 86.925)
+		(width 0.6)
+		(layer "F.Cu")
+		(net "+5V")
+	)
 	(via
 		(at 175.54 87.95)
@@
 		(net "/Screen_DC")
 	)
+	(segment
+		(start 126.345 94.13)
+		(end 123.67 94.13)
+		(width 0.3)
+		(layer "F.Cu")
+		(net "/Screen_DC")
+	)
 	(via
 		(at 130.095 90.38)
@@
 		(start 145.188603 91.9)
 		(end 144.645001 91.9)
-		(width 0.3)
+		(width 0.2)
 		(layer "B.Cu")
 		(net "/D-")
 	)
 	(segment
-		(start 144.235001 91.49)
-		(end 143.11 91.49)
-		(width 0.3)
+		(start 148.02 89.068603)
+		(end 145.188603 91.9)
+		(width 0.2)
 		(layer "B.Cu")
 		(net "/D-")
 	)
 	(segment
-		(start 148.02 87.805)
-		(end 148.02 89.068603)
-		(width 0.3)
+		(start 144.645001 91.9)
+		(end 144.235001 91.49)
+		(width 0.2)
 		(layer "B.Cu")
 		(net "/D-")
 	)
 	(segment
-		(start 148.02 89.068603)
-		(end 145.188603 91.9)
-		(width 0.3)
+		(start 148.02 87.805)
+		(end 148.02 89.068603)
+		(width 0.2)
 		(layer "B.Cu")
 		(net "/D-")
 	)
 	(segment
-		(start 144.645001 91.9)
-		(end 144.235001 91.49)
-		(width 0.3)
+		(start 144.235001 91.49)
+		(end 143.11 91.49)
+		(width 0.2)
 		(layer "B.Cu")
 		(net "/D-")
 	)
 	(segment
-		(start 149.92 87.805)
-		(end 149.57 88.155)
-		(width 0.3)
+		(start 149.289842 88.7175)
+		(end 149.0075 88.7175)
+		(width 0.2)
 		(layer "B.Cu")
 		(net "/D+")
 	)
 	(segment
-		(start 149.310552 88.7675)
-		(end 148.9575 88.7675)
-		(width 0.3)
+		(start 145.375 92.35)
+		(end 144.645001 92.35)
+		(width 0.2)
 		(layer "B.Cu")
 		(net "/D+")
 	)
 	(segment
-		(start 149.57 88.155)
-		(end 149.57 88.508052)
-		(width 0.3)
+		(start 149.52 88.487342)
+		(end 149.289842 88.7175)
+		(width 0.2)
 		(layer "B.Cu")
 		(net "/D+")
 	)
 	(segment
-		(start 149.57 88.508052)
-		(end 149.310552 88.7675)
-		(width 0.3)
+		(start 149.52 88.205)
+		(end 149.52 88.487342)
+		(width 0.2)
 		(layer "B.Cu")
 		(net "/D+")
 	)
 	(segment
-		(start 148.9575 88.7675)
-		(end 145.375 92.35)
-		(width 0.3)
+		(start 144.645001 92.35)
+		(end 144.235001 92.76)
+		(width 0.2)
 		(layer "B.Cu")
 		(net "/D+")
 	)
 	(segment
-		(start 144.235001 92.76)
-		(end 143.11 92.76)
-		(width 0.3)
+		(start 149.92 87.805)
+		(end 149.52 88.205)
+		(width 0.2)
 		(layer "B.Cu")
 		(net "/D+")
 	)
 	(segment
-		(start 145.375 92.35)
-		(end 144.645001 92.35)
-		(width 0.3)
+		(start 149.0075 88.7175)
+		(end 145.375 92.35)
+		(width 0.2)
 		(layer "B.Cu")
 		(net "/D+")
 	)
 	(segment
-		(start 144.645001 92.35)
-		(end 144.235001 92.76)
-		(width 0.3)
+		(start 144.235001 92.76)
+		(end 143.11 92.76)
+		(width 0.2)
 		(layer "B.Cu")
 		(net "/D+")
